File: plate_kicad_files/jiu_plate.kicad_pcb (KiCad board)
At the start: 2 copper layers, 304.8 x 105.4 mm, 0 parts

Commit message: gitignore, stab orientation
- Added backup files to gitignore
- Fix enter, right shift keys stab orientations
- New KiCAD version
Other:
- outline, holes or cut-outs redrawn
